Commit message: port f1tenth_gym_ros to here, adding namespace support for topic and robot description and other configs

File: nturt_nms1_description/urdf/lidar.xacro (robot description, xacro)
@@ -1,5 +1,5 @@
 <?xml version="1.0"?>
 <robot xmlns:xacro="http://www.ros.org/wiki/xacro">
-<!-- default argument -->
+    <!-- default argument -->
     <xacro:arg name="using_gazebo" default="false"/>
     <!-- include macro from other files-->
@@ -15,29 +15,29 @@
                     <update_rate>5</update_rate>
                     <ray>
-                    <scan>
-                        <horizontal>
-                        <samples>360</samples>
-                        <resolution>1.0</resolution>
-                        <min_angle>0.0</min_angle>
-                        <max_angle>6.28</max_angle>
-                        </horizontal>
-                    </scan>
-                    <range>
-                        <min>0.12</min>
-                        <max>3.5</max>
-                        <resolution>0.015</resolution>
-                    </range>
-                    <noise>
-                        <type>gaussian</type>
-                        <mean>0.0</mean>
-                        <stddev>0.01</stddev>
-                    </noise>
+                        <scan>
+                            <horizontal>
+                            <samples>360</samples>
+                            <resolution>1.0</resolution>
+                            <min_angle>0.0</min_angle>
+                            <max_angle>6.28</max_angle>
+                            </horizontal>
+                        </scan>
+                        <range>
+                            <min>0.12</min>
+                            <max>3.5</max>
+                            <resolution>0.015</resolution>
+                        </range>
+                        <noise>
+                            <type>gaussian</type>
+                            <mean>0.0</mean>
+                            <stddev>0.01</stddev>
+                        </noise>
                     </ray>
                     <plugin name="scan" filename="libgazebo_ros_ray_sensor.so">
-                    <ros>
-                        <remapping>~/out:=scan</remapping>
-                    </ros>
-                    <output_type>sensor_msgs/LaserScan</output_type>
-                    <frame_name>${name}</frame_name>
+                        <ros>
+                            <remapping>~/out:=scan</remapping>
+                        </ros>
+                        <output_type>sensor_msgs/LaserScan</output_type>
+                        <frame_name>${name}</frame_name>
                     </plugin>
                 </sensor>

File: nturt_nms1_description/urdf/nms1.xacro (robot description, xacro)
@@ -1,4 +1,6 @@
 <?xml version="1.0"?>
 <robot name="nms1" xmlns:xacro="http://www.ros.org/wiki/xacro">
+    <!-- default argument -->
+    <xacro:arg name="ns" default=""/>
     <!-- include macro from other files-->
     <xacro:include filename="$(find nturt_nms1_description)/urdf/lidar.xacro"/>
@@ -12,53 +14,66 @@
     <!-- wheel macro -->
     <xacro:macro name="wheel" params="name">
+        <link name="${name}_axle"/>
         <xacro:solid_cylinder name="${name}" length="0.05" radius="0.06" rpy="${radians(90)} 0 0" mass="0.05" material="Black"/>
+        <joint name="${name}_drive_joint" type="continuous">
+            <parent link="${name}_axle"/>
+            <child link="${name}"/>
+            <axis xyz="0 1 0"/>
+        </joint>
+    </xacro:macro>
+    <!-- steering wheel macro -->
+    <xacro:macro name="steering_wheel" params="name">
+        <link name="${name}_steering_hinge"/>
+        <xacro:wheel name="${name}"/>
+        <joint name="${name}_steering_joint" type="revolute">
+            <parent link="${name}_steering_hinge"/>
+            <child link="${name}_axle"/>
+            <axis xyz="0 0 1"/>
+            <limit lower="${radians(-30)}" upper="${radians(30)}" effort="10000000" velocity="1000000"/>
+        </joint>
     </xacro:macro>
     <!-- robot definition -->
-    <link name="base_link"/>
-    <link name="base_footprint"/>
-    <xacro:chassis name="chassis"/>
-    <xacro:lidar name="lidar"/>
-    <xacro:wheel name="front_left_wheel"/>
-    <xacro:wheel name="front_right_wheel"/>
-    <xacro:wheel name="rear_left_wheel"/>
-    <xacro:wheel name="rear_right_wheel"/>
-    <joint name="base_joint" type="fixed">
-        <parent link="base_link"/>
-        <child link="base_footprint"/>
+    <link name="$(arg ns)/base_link"/>
+    <link name="$(arg ns)/base_footprint"/>
+    <xacro:chassis name="$(arg ns)/chassis"/>
+    <xacro:lidar name="$(arg ns)/lidar"/>
+    <xacro:steering_wheel name="$(arg ns)/front_left_wheel"/>
+    <xacro:steering_wheel name="$(arg ns)/front_right_wheel"/>
+    <xacro:wheel name="$(arg ns)/rear_left_wheel"/>
+    <xacro:wheel name="$(arg ns)/rear_right_wheel"/>
+    <joint name="$(arg ns)/base_footprint_mount" type="fixed">
+        <parent link="$(arg ns)/base_link"/>
+        <child link="$(arg ns)/base_footprint"/>
         <origin xyz="0.0 0.0 -0.1" rpy="0 0 0"/>
     </joint>
-    <joint name="base_link" type="fixed">
-        <parent link="base_link"/>
-        <child link="chassis"/>
+    <joint name="$(arg ns)/base_mount" type="fixed">
+        <parent link="$(arg ns)/base_link"/>
+        <child link="$(arg ns)/chassis"/>
         <origin xyz="0 0 0" rpy="0 0 0"/>
     </joint>
-    <joint name="lidar_joint" type="fixed">
-        <parent link="chassis"/>
-        <child link="lidar"/>
+    <joint name="$(arg ns)/lidar_mount" type="fixed">
+        <parent link="$(arg ns)/chassis"/>
+        <child link="$(arg ns)/lidar"/>
         <origin xyz="0.15 0 0.05" rpy="0 0 0"/>
     </joint>
-    <joint name="front_left_wheel_joint" type="continuous">
-        <parent link="chassis"/>
-        <child link="front_left_wheel"/>
+    <joint name="$(arg ns)/front_left_wheel_mount" type="fixed">
+        <parent link="$(arg ns)/chassis"/>
+        <child link="$(arg ns)/front_left_wheel_steering_hinge"/>
         <origin xyz="0.2 -0.15 -0.04" rpy="0 0 0"/>
-        <axis xyz="0 1 0"/>
     </joint>
-    <joint name="front_right_wheel_joint" type="continuous">
-        <parent link="chassis"/>
-        <child link="front_right_wheel"/>
+    <joint name="$(arg ns)/front_right_wheel_mount" type="fixed">
+        <parent link="$(arg ns)/chassis"/>
+        <child link="$(arg ns)/front_right_wheel_steering_hinge"/>
         <origin xyz="0.2 0.15 -0.04" rpy="0 0 0"/>
-        <axis xyz="0 1 0"/>
     </joint>
-    <joint name="rear_left_wheel_joint" type="continuous">
-        <parent link="chassis"/>
-        <child link="rear_left_wheel"/>
+    <joint name="$(arg ns)/rear_left_wheel_mount" type="fixed">
+        <parent link="$(arg ns)/chassis"/>
+        <child link="$(arg ns)/rear_left_wheel_axle"/>
         <origin xyz="-0.2 -0.15 -0.04" rpy="0 0 0"/>
-        <axis xyz="0 1 0"/>
     </joint>
-    <joint name="rear_right_wheel_joint" type="continuous">
-        <parent link="chassis"/>
-        <child link="rear_right_wheel"/>
+    <joint name="$(arg ns)/rear_right_wheel_mount" type="fixed">
+        <parent link="$(arg ns)/chassis"/>
+        <child link="$(arg ns)/rear_right_wheel_axle"/>
         <origin xyz="-0.2 0.15 -0.04" rpy="0 0 0"/>
-        <axis xyz="0 1 0"/>
     </joint>
     <xacro:ros2_control/>

Commit message: move f1tenth_gym to its own package and adding controllers

File: nturt_nms1_description/urdf/lidar.xacro (robot description, xacro)
@@ -4,8 +4,9 @@
     <xacro:arg name="using_gazebo" default="false"/>
     <!-- include macro from other files-->
+    <xacro:include filename="$(find nturt_nms1_description)/urdf/properties.xacro"/>
     <xacro:include filename="$(find nturt_nms1_description)/urdf/simple_geometry.xacro"/>
     <!-- lidar macro-->
     <xacro:macro name="lidar" params="name">
-        <xacro:solid_cylinder name="${name}" length="0.05" radius="0.05" xyz="0 0 0.025" mass="0.05" material="Red"/>
+        <xacro:solid_cylinder name="${name}" length="0.05" radius="0.05" xyz="0 0 0.025" mass="${lidar_mass}" material="Red"/>
         <xacro:if value="$(arg using_gazebo)">
             <gazebo reference="${name}">

File: nturt_nms1_description/urdf/nms1.xacro (robot description, xacro)
@@ -2,78 +2,84 @@
 <robot name="nms1" xmlns:xacro="http://www.ros.org/wiki/xacro">
     <!-- default argument -->
-    <xacro:arg name="ns" default=""/>
+    <xacro:arg name="namespace" default=""/>
+    <!-- constant definition -->
+    <xacro:property name="empty" value=""/>
+    <xacro:if value="${'$(arg namespace)' != ''}">
+        <xacro:property name="link_prefix" value="$(arg namespace)/"/>
+    </xacro:if>
+    <xacro:unless value="${'$(arg namespace)' != ''}">
+        <xacro:property name="link_prefix" value=""/>
+    </xacro:unless>
     <!-- include macro from other files-->
     <xacro:include filename="$(find nturt_nms1_description)/urdf/lidar.xacro"/>
     <xacro:include filename="$(find nturt_nms1_description)/urdf/material.xacro"/>
+    <xacro:include filename="$(find nturt_nms1_description)/urdf/properties.xacro"/>
     <xacro:include filename="$(find nturt_nms1_description)/urdf/ros2_control.xacro"/>
     <xacro:include filename="$(find nturt_nms1_description)/urdf/simple_geometry.xacro"/>
     <!-- chassis macro -->
     <xacro:macro name="chassis" params="name">
-        <xacro:solid_cuboid name="${name}" length="0.4" width="0.2" hight="0.10" mass="2" material="Blue"/>
+        <xacro:solid_cuboid name="${name}" length="${chassis_length}" width="${chassis_width}" height="${chassis_height}" mass="${chassis_mass}" material="Blue"/>
     </xacro:macro>
     <!-- wheel macro -->
-    <xacro:macro name="wheel" params="name">
+    <xacro:macro name="wheel" params="name drive_mimic:=${empty}">
         <link name="${name}_axle"/>
-        <xacro:solid_cylinder name="${name}" length="0.05" radius="0.06" rpy="${radians(90)} 0 0" mass="0.05" material="Black"/>
+        <xacro:solid_cylinder name="${name}" length="${wheel_width}" radius="${wheel_radius}" rpy="${radians(90)} 0 0" mass="${wheel_mass}" material="Black"/>
         <joint name="${name}_drive_joint" type="continuous">
             <parent link="${name}_axle"/>
             <child link="${name}"/>
             <axis xyz="0 1 0"/>
+            <xacro:if value="${drive_mimic != ''}">
+                <mimic joint="${drive_mimic}_drive_joint" multiplier="1" offset="0"/>
+            </xacro:if>
         </joint>
     </xacro:macro>
     <!-- steering wheel macro -->
-    <xacro:macro name="steering_wheel" params="name">
+    <xacro:macro name="steering_wheel" params="name drive_mimic:=${empty}">
         <link name="${name}_steering_hinge"/>
-        <xacro:wheel name="${name}"/>
+        <xacro:wheel name="${name}" drive_mimic="${drive_mimic}"/>
         <joint name="${name}_steering_joint" type="revolute">
             <parent link="${name}_steering_hinge"/>
             <child link="${name}_axle"/>
             <axis xyz="0 0 1"/>
-            <limit lower="${radians(-30)}" upper="${radians(30)}" effort="10000000" velocity="1000000"/>
+            <limit lower="${-steering_limit}" upper="${steering_limit}" effort="10000000" velocity="1000000"/>
         </joint>
     </xacro:macro>
     <!-- robot definition -->
-    <link name="$(arg ns)/base_link"/>
-    <link name="$(arg ns)/base_footprint"/>
-    <xacro:chassis name="$(arg ns)/chassis"/>
-    <xacro:lidar name="$(arg ns)/lidar"/>
-    <xacro:steering_wheel name="$(arg ns)/front_left_wheel"/>
-    <xacro:steering_wheel name="$(arg ns)/front_right_wheel"/>
-    <xacro:wheel name="$(arg ns)/rear_left_wheel"/>
-    <xacro:wheel name="$(arg ns)/rear_right_wheel"/>
-    <joint name="$(arg ns)/base_footprint_mount" type="fixed">
-        <parent link="$(arg ns)/base_link"/>
-        <child link="$(arg ns)/base_footprint"/>
-        <origin xyz="0.0 0.0 -0.1" rpy="0 0 0"/>
+    <link name="${link_prefix}base_link"/>
+    <xacro:chassis name="${link_prefix}chassis"/>
+    <xacro:lidar name="${link_prefix}laser"/>
+    <xacro:steering_wheel name="${link_prefix}front_left_wheel" drive_mimic="${link_prefix}rear_left_wheel"/>
+    <xacro:steering_wheel name="${link_prefix}front_right_wheel" drive_mimic="${link_prefix}rear_right_wheel"/>
+    <xacro:wheel name="${link_prefix}rear_left_wheel"/>
+    <xacro:wheel name="${link_prefix}rear_right_wheel"/>
+    <joint name="${link_prefix}base_mount" type="fixed">
+        <parent link="${link_prefix}base_link"/>
+        <child link="${link_prefix}chassis"/>
+        <origin xyz="0 0 ${chassis_vertical_offset}" rpy="0 0 0"/>
     </joint>
-    <joint name="$(arg ns)/base_mount" type="fixed">
-        <parent link="$(arg ns)/base_link"/>
-        <child link="$(arg ns)/chassis"/>
-        <origin xyz="0 0 0" rpy="0 0 0"/>
+    <joint name="${link_prefix}laser_mount" type="fixed">
+        <parent link="${link_prefix}chassis"/>
+        <child link="${link_prefix}laser"/>
+        <origin xyz="${lidar_longitudinal_offset} 0 ${lidar_vertical_offset}" rpy="0 0 0"/>
     </joint>
-    <joint name="$(arg ns)/lidar_mount" type="fixed">
-        <parent link="$(arg ns)/chassis"/>
-        <child link="$(arg ns)/lidar"/>
-        <origin xyz="0.15 0 0.05" rpy="0 0 0"/>
+    <joint name="${link_prefix}front_left_wheel_mount" type="fixed">
+        <parent link="${link_prefix}chassis"/>
+        <child link="${link_prefix}front_left_wheel_steering_hinge"/>
+        <origin xyz="${wheel_longitudinal_offset} -${wheel_lateral_offset} -${wheel_vertical_offset}" rpy="0 0 0"/>
     </joint>
-    <joint name="$(arg ns)/front_left_wheel_mount" type="fixed">
-        <parent link="$(arg ns)/chassis"/>
-        <child link="$(arg ns)/front_left_wheel_steering_hinge"/>
-        <origin xyz="0.2 -0.15 -0.04" rpy="0 0 0"/>
+    <joint name="${link_prefix}front_right_wheel_mount" type="fixed">
+        <parent link="${link_prefix}chassis"/>
+        <child link="${link_prefix}front_right_wheel_steering_hinge"/>
+        <origin xyz="${wheel_longitudinal_offset} ${wheel_lateral_offset} -${wheel_vertical_offset}" rpy="0 0 0"/>
     </joint>
-    <joint name="$(arg ns)/front_right_wheel_mount" type="fixed">
-        <parent link="$(arg ns)/chassis"/>
-        <child link="$(arg ns)/front_right_wheel_steering_hinge"/>
-        <origin xyz="0.2 0.15 -0.04" rpy="0 0 0"/>
+    <joint name="${link_prefix}rear_left_wheel_mount" type="fixed">
+        <parent link="${link_prefix}chassis"/>
+        <child link="${link_prefix}rear_left_wheel_axle"/>
+        <origin xyz="-${wheel_longitudinal_offset} -${wheel_lateral_offset} -${wheel_vertical_offset}" rpy="0 0 0"/>
     </joint>
-    <joint name="$(arg ns)/rear_left_wheel_mount" type="fixed">
-        <parent link="$(arg ns)/chassis"/>
-        <child link="$(arg ns)/rear_left_wheel_axle"/>
-        <origin xyz="-0.2 -0.15 -0.04" rpy="0 0 0"/>
-    </joint>
-    <joint name="$(arg ns)/rear_right_wheel_mount" type="fixed">
-        <parent link="$(arg ns)/chassis"/>
-        <child link="$(arg ns)/rear_right_wheel_axle"/>
-        <origin xyz="-0.2 0.15 -0.04" rpy="0 0 0"/>
+    <joint name="${link_prefix}rear_right_wheel_mount" type="fixed">
+        <parent link="${link_prefix}chassis"/>
+        <child link="${link_prefix}rear_right_wheel_axle"/>
+        <origin xyz="-${wheel_longitudinal_offset} ${wheel_lateral_offset} -${wheel_vertical_offset}" rpy="0 0 0"/>
     </joint>
     <xacro:ros2_control/>

File: nturt_nms1_description/urdf/ros2_control.xacro (robot description, xacro)
@@ -3,22 +3,29 @@
     <!-- default argument -->
     <xacro:arg name="using_gazebo" default="false"/>
-    <!-- wheel control config macro -->
-    <xacro:macro name="wheel_control_config" params="wheel_name">
-        <joint name="${wheel_name}">
-            <command_interface name="position"/>
+    <xacro:arg name="using_fake_hardware" default="false"/>
+    <!-- include macro from other files-->
+    <xacro:include filename="$(find nturt_nms1_description)/urdf/properties.xacro"/>
+    <!-- steering_wheel_control_config macro -->
+    <xacro:macro name="steering_wheel_control_config" params="name">
+        <joint name="${name}">
+            <command_interface name="position">
+                <param name="min">-${steering_limit}</param>
+                <param name="max">${steering_limit}</param>
+            </command_interface>
+            <state_interface name="position"/>
+        </joint>
+    </xacro:macro>
+    <!-- drive_wheel_control_config macro -->
+    <xacro:macro name="drive_wheel_control_config" params="name">
+        <joint name="${name}">
             <command_interface name="velocity">
-                <param name="min">-1</param>
-                <param name="max">1</param>
-            </command_interface>
-            <command_interface name="acceleration">
-                <param name="min">-10</param>
-                <param name="max">10</param>
+                <param name="min">-${max_speed}</param>
+                <param name="max">${max_speed}</param>
             </command_interface>
             <state_interface name="position"/>
             <state_interface name="velocity"/>
-            <state_interface name="acceleration"/>
         </joint>
     </xacro:macro>
-    <!-- nms1 ros2_control macro -->
+    <!-- ros2_control macro -->
     <xacro:macro name="ros2_control">
         <ros2_control name="car_control_system" type="system">
@@ -29,9 +36,16 @@
             </xacro:if>
             <xacro:unless value="$(arg using_gazebo)">
+                <xacro:if value="$(arg using_fake_hardware)">
+                    <hardware>
+                        <plugin>mock_components/GenericSystem</plugin>
+                    </hardware>
+                </xacro:if>
+                <xacro:unless value="$(arg using_fake_hardware)">
+                </xacro:unless>
             </xacro:unless>
-            <xacro:wheel_control_config wheel_name="front_left_wheel_joint"/>
-            <xacro:wheel_control_config wheel_name="front_right_wheel_joint"/>
-            <xacro:wheel_control_config wheel_name="rear_left_wheel_joint"/>
-            <xacro:wheel_control_config wheel_name="rear_right_wheel_joint"/>
+            <xacro:steering_wheel_control_config name="front_left_wheel_steering_joint"/>
+            <xacro:steering_wheel_control_config name="front_right_wheel_steering_joint"/>
+            <xacro:drive_wheel_control_config name="rear_left_wheel_drive_joint"/>
+            <xacro:drive_wheel_control_config name="rear_right_wheel_drive_joint"/>
         </ros2_control>
         <xacro:if value="$(arg using_gazebo)">

File: nturt_nms1_description/urdf/simple_geometry.xacro (robot description, xacro)
@@ -6,6 +6,6 @@
     <!-- constant definition -->
     <xacro:property name="triple_zero" value="0 0 0"/>
-    <!-- solid cuboid property macro -->
-    <xacro:macro name="solid_cuboid" params="name length width hight xyz:=${triple_zero} rpy:=${triple_zero} mass:=1 material:=White">
+    <!-- solid_cuboid macro -->
+    <xacro:macro name="solid_cuboid" params="name length width height xyz:=${triple_zero} rpy:=${triple_zero} mass:=1 material:=White">
         <link name="${name}">
             <inertial>
@@ -13,6 +13,6 @@
                 <mass value="${mass}"/>
                 <inertia
-                    ixx="${1 / 12 * mass * (width ** 2 + hight ** 2)}"
-                    iyy="${1 / 12 * mass * (length ** 2 + hight ** 2)}"
+                    ixx="${1 / 12 * mass * (width ** 2 + height ** 2)}"
+                    iyy="${1 / 12 * mass * (length ** 2 + height ** 2)}"
                     izz="${1 / 12 * mass * (length ** 2 + width ** 2)}"
                     ixy="0.0"
@@ -24,5 +24,5 @@
                 <origin xyz="${xyz}" rpy="${rpy}"/>
                 <geometry>
-                    <box size="${length} ${width} ${hight}"/>
+                    <box size="${length} ${width} ${height}"/>
                 </geometry>
                 <material name="${material}"/>
@@ -31,5 +31,5 @@
                 <origin xyz="${xyz}" rpy="${rpy}"/>
                 <geometry>
-                    <box size="${length} ${width} ${hight}"/>
+                    <box size="${length} ${width} ${height}"/>
                 </geometry>
             </collision>
@@ -42,5 +42,5 @@
         </xacro:if>
     </xacro:macro>
-    <!-- solid cylinder property macro -->
+    <!-- solid_cylinder macro -->
     <xacro:macro name="solid_cylinder" params="name length radius xyz:=${triple_zero} rpy:=${triple_zero} mass:=1 material:=White">
         <link name="${name}">
@@ -78,5 +78,5 @@
         </xacro:if>
     </xacro:macro>
-    <!-- solid sphere property macro -->
+    <!-- solid_sphere macro -->
     <xacro:macro name="soild_sphere" params="name radius xyz:=${triple_zero} mass:=1 material:=White">
         <link name="${name}">
